Commit message: Put macros in separate files, add LiDAR sensor, add gz_bridge.yaml, add gazebo_launch.py to launch Gazebo and spawn robot

File: ros2/palmbot_description/urdf/palmbot_description.xacro (robot description, xacro)
@@ -1,4 +1,6 @@
 <?xml version="1.0"?>
 <robot name="palmbot" xmlns:xacro="http://ros.org/wiki/xacro">
+  <xacro:include filename="inertial_macros.xacro"/>
+  <xacro:include filename="wheel.xacro"/>
   <!-- Robot Constants -->
   <xacro:property name="base_width" value="0.070"/>
@@ -13,25 +15,4 @@
   <xacro:property name="wheel_xoff" value="0.014"/>
   <xacro:property name="caster_xoff" value="0.029"/>
-  <!-- Define inertial property macros  -->
-  <xacro:macro name="box_inertia" params="m w h d">
-    <inertial>
-      <origin xyz="0 0 0" rpy="${pi/2} 0 ${pi/2}"/>
-      <mass value="${m}"/>
-      <inertia ixx="${(m/12) * (h*h + d*d)}" ixy="0.0" ixz="0.0" iyy="${(m/12) * (w*w + d*d)}" iyz="0.0" izz="${(m/12) * (w*w + h*h)}"/>
-    </inertial>
-  </xacro:macro>
-  <xacro:macro name="cylinder_inertia" params="m r h">
-    <inertial>
-      <origin xyz="0 0 0" rpy="${pi/2} 0 0" />
-      <mass value="${m}"/>
-      <inertia ixx="${(m/12) * (3*r*r + h*h)}" ixy = "0" ixz = "0" iyy="${(m/12) * (3*r*r + h*h)}" iyz = "0" izz="${(m/2) * (r*r)}"/>
-    </inertial>
-  </xacro:macro>
-  <xacro:macro name="sphere_inertia" params="m r">
-    <inertial>
-      <mass value="${m}"/>
-      <inertia ixx="${(2/5) * m * (r*r)}" ixy="0.0" ixz="0.0" iyy="${(2/5) * m * (r*r)}" iyz="0.0" izz="${(2/5) * m * (r*r)}"/>
-    </inertial>
-  </xacro:macro>
   <!-- Robot Footprint -->
   <link name="base_footprint"/>
@@ -59,5 +40,5 @@
   </joint>
   <!-- LiDAR -->
-  <link name="lidar">
+  <link name="lidar_link">
     <visual>
       <geometry>
@@ -74,38 +55,41 @@
       </geometry>
     </collision>
-    <xacro:cylinder_inertia m="0.05" r="${lidar_radius}" h="${lidar_height}"/>
+    <xacro:cylinder_inertia m="0.05" r="${lidar_radius}" h="${lidar_height}">
+      <origin xyz="0 0 0" rpy="0 0 0"/>
+    </xacro:cylinder_inertia>
   </link>
   <joint name="lidar_joint" type="fixed">
     <parent link="base_link"/>
-    <child link="lidar"/>
+    <child link="lidar_link"/>
     <origin xyz="0.0 0.0 ${base_height/2+lidar_height/2}" rpy="0 0 0"/>
   </joint>
+  <gazebo reference="lidar_link">
+    <sensor name="lidar" type="gpu_lidar">
+      <pose> 0 0 0 0 0 0 </pose>
+      <visualize>true</visualize>
+      <update_rate>10</update_rate>
+      <lidar>
+        <scan>
+          <horizontal>
+            <samples>450</samples>
+            <min_angle>${-pi}</min_angle>
+            <max_angle>${pi}</max_angle>
+          </horizontal>
+        </scan>
+        <range>
+          <min>0.02</min>
+          <max>12</max>
+        </range>
+      </lidar>
+      <noise>
+        <type>gaussian</type>
+        <mean>0.0</mean>
+        <stddev>0.01</stddev>
+      </noise>
+      <topic>scan</topic>
+      <gz_frame_id>lidar_link</gz_frame_id>
+    </sensor>
+  </gazebo>
   <!-- Wheels -->
-  <xacro:macro name="wheel" params="prefix x_reflect y_reflect">
-    <link name="${prefix}_link">
-      <visual>
-        <origin xyz="0 0 0" rpy="${pi/2} 0 0"/>
-        <geometry>
-            <cylinder radius="${wheel_radius}" length="${wheel_width}"/>
-        </geometry>
-        <material name="White">
-          <color rgba="1.0 1.0 1.0 1.0"/>
-        </material>
-      </visual>
-      <collision>
-        <origin xyz="0 0 0" rpy="${pi/2} 0 0"/>
-        <geometry>
-          <cylinder radius="${wheel_radius}" length="${wheel_width}"/>
-        </geometry>
-      </collision>
-      <xacro:cylinder_inertia m="0.005" r="${wheel_radius}" h="${wheel_width}"/>
-    </link>
-    <joint name="${prefix}_joint" type="continuous">
-      <parent link="base_link"/>
-      <child link="${prefix}_link"/>
-      <origin xyz="${x_reflect*wheel_xoff} ${y_reflect*(base_width/2+wheel_width/2+wheel_ygap)} ${-wheel_zoff}" rpy="0 0 0"/>
-      <axis xyz="0 1 0"/>
-    </joint>
-  </xacro:macro>
   <xacro:wheel prefix="drivewhl_l" x_reflect="-1" y_reflect="1" />
   <xacro:wheel prefix="drivewhl_r" x_reflect="-1" y_reflect="-1" />
@@ -141,3 +125,16 @@
     <slip2 value="1.0"/>
   </gazebo>
+  <!-- DiffDrive Plugin -->
+  <gazebo>
+    <plugin
+      filename="gz-sim-diff-drive-system"
+      name="gz::sim::systems::DiffDrive">
+      <left_joint>drivewhl_l_joint</left_joint>
+      <right_joint>drivewhl_r_joint</right_joint>
+      <wheel_separation>${base_width+2*wheel_ygap+wheel_width}</wheel_separation>
+      <wheel_radius>${wheel_radius}</wheel_radius>
+      <odom_publish_frequency>1</odom_publish_frequency>
+      <topic>cmd_vel</topic>
+    </plugin>
+  </gazebo>
 </robot>

Commit message: Add IMU and custom world

File: ros2/palmbot_description/urdf/palmbot_description.xacro (robot description, xacro)
@@ -2,5 +2,5 @@
 <robot name="palmbot" xmlns:xacro="http://ros.org/wiki/xacro">
   <xacro:include filename="inertial_macros.xacro"/>
-  <xacro:include filename="wheel.xacro"/>
+  <xacro:include filename="wheel_macro.xacro"/>
   <!-- Robot Constants -->
   <xacro:property name="base_width" value="0.070"/>
@@ -15,4 +15,5 @@
   <xacro:property name="wheel_xoff" value="0.014"/>
   <xacro:property name="caster_xoff" value="0.029"/>
+  <xacro:property name="imu_zoff" value="0.0091"/>
   <!-- Robot Footprint -->
   <link name="base_footprint"/>
@@ -37,5 +38,5 @@
     <parent link="base_footprint"/>
     <child link="base_link"/>
-    <origin xyz="0.0 0.0 ${wheel_radius+wheel_zoff}" rpy="0 0 0"/>
+    <origin xyz="${wheel_xoff} 0.0 ${wheel_radius+wheel_zoff}" rpy="0 0 0"/>
   </joint>
   <!-- LiDAR -->
@@ -91,4 +92,68 @@
     </sensor>
   </gazebo>
+  <!-- IMU -->
+  <link name="imu_link">
+    <visual>
+      <geometry>
+        <box size="0.0025 0.003 0.00083"/>
+      </geometry>
+    </visual>
+  </link>
+  <joint name="imu_joint" type="fixed">
+    <parent link="base_link"/>
+    <child link="imu_link"/>
+    <origin xyz="${-wheel_xoff} 0.0 ${-imu_zoff+0.000415}" rpy="0 0 0"/>
+  </joint>
+  <gazebo reference="imu_link">
+    <sensor name="imu" type="imu">
+      <always_on>1</always_on>
+      <update_rate>208</update_rate>
+      <visualize>true</visualize>
+      <imu>
+        <angular_velocity>
+          <x>
+            <noise type="gaussian">
+              <mean>0.0</mean>
+              <stddev>1.3e-3</stddev>
+            </noise>
+          </x>
+          <y>
+            <noise type="gaussian">
+              <mean>0.0</mean>
+              <stddev>1.3e-3</stddev>
+            </noise>
+          </y>
+          <z>
+            <noise type="gaussian">
+              <mean>0.0</mean>
+              <stddev>1.3e-3</stddev>
+            </noise>
+          </z>
+        </angular_velocity>
+        <linear_acceleration>
+          <x>
+            <noise type="gaussian">
+              <mean>0.0</mean>
+              <stddev>1.3e-2</stddev>
+            </noise>
+          </x>
+          <y>
+            <noise type="gaussian">
+              <mean>0.0</mean>
+              <stddev>1.3e-2</stddev>
+            </noise>
+          </y>
+          <z>
+            <noise type="gaussian">
+              <mean>0.0</mean>
+              <stddev>1.3e-2</stddev>
+            </noise>
+          </z>
+        </linear_acceleration>
+      </imu>
+      <topic>imu</topic>
+      <gz_frame_id>imu_link</gz_frame_id>
+    </sensor>
+  </gazebo>
   <!-- Wheels -->
   <xacro:wheel prefix="drivewhl_l" x_reflect="-1" y_reflect="1" />
@@ -134,6 +199,9 @@
       <wheel_separation>${base_width+2*wheel_ygap+wheel_width}</wheel_separation>
       <wheel_radius>${wheel_radius}</wheel_radius>
-      <odom_publish_frequency>1</odom_publish_frequency>
+      <odom_publish_frequency>30</odom_publish_frequency>
       <topic>cmd_vel</topic>
+      <frame_id>odom</frame_id>
+      <child_frame_id>base_footprint</child_frame_id>
+      <odom_topic>odometry</odom_topic>
     </plugin>
   </gazebo>
